Commit message: enabled self collisions

File: urdfs/spider_bot_v0.urdf (robot description, URDF)
Before this commit: robot spiderbot, 13 links, 12 joints
Links:
- link BL1: geometry collision box size=0.127 0.6541 0.381; visual box size=0.127 0.6541 0.381
- link BR1: geometry collision box size=0.127 0.6541 0.381; visual box size=0.127 0.6541 0.381
- link FL1: geometry collision box size=0.127 0.6541 0.381; visual box size=0.127 0.6541 0.381
- link FR1: geometry collision box size=0.127 0.6541 0.381; visual box size=0.127 0.6541 0.381
- link SpiderBody: mass 5 -> 25

Commit message: Adjusted urdf (main body height and leg range)

File: urdfs/spider_bot_v0.urdf (robot description, URDF)
Before this commit: robot spiderbot, 13 links, 12 joints
Links:
- link SpiderBody: geometry collision box size=0.95 0.93 0.89; visual box size=0.95 0.93 0.89
Joints:
- joint BLJ2: limit lower=-1.571 upper=1.571 effort=100 velocity=100 -> lower=-1.571 upper=-0.4 effort=100 velocity=100
- joint BRJ2: limit lower=-1.571 upper=1.571 effort=100 velocity=100 -> lower=-1.571 upper=-0.4 effort=100 velocity=100
- joint FLJ2: limit lower=-1.571 upper=1.571 effort=100 velocity=100 -> lower=-1.571 upper=-0.4 effort=100 velocity=100
- joint FRJ2: limit lower=-1.571 upper=1.571 effort=100 velocity=100 -> lower=-1.571 upper=-0.4 effort=100 velocity=100

Commit message: Modified legs to hopefully allow for rubber ends

File: urdfs/spider_bot_v0.urdf (robot description, URDF)
Before this commit: robot spiderbot, 13 links, 12 joints
Links:
- added link BLE, mass 0.5; collision sphere radius=0.08; visual sphere radius=0.08
- added link BRE, mass 0.5; collision sphere radius=0.08; visual sphere radius=0.08
- added link FLE, mass 0.5; collision sphere radius=0.08; visual sphere radius=0.08
- added link FRE, mass 0.5; collision sphere radius=0.08; visual sphere radius=0.08
- link BL2: geometry collision cylinder length=1.04 radius=.08; visual cylinder length=1.04 radius=.08
- link BR2: geometry collision cylinder length=1.04 radius=.08; visual cylinder length=1.04 radius=.08
- link FL2: geometry collision cylinder length=1.04 radius=.08; visual cylinder length=1.04 radius=.08
- link FR2: geometry collision cylinder length=1.04 radius=.08; visual cylinder length=1.04 radius=.08
Joints:
- added joint BLEJ: type fixed, parent BL2, child BLE, origin xyz=0.0 1.04 0.0 rpy=0.0 0.0 0.0
- added joint BREJ: type fixed, parent BR2, child BRE, origin xyz=0.0 1.04 0.0 rpy=0.0 0.0 0.0
- added joint FLEJ: type fixed, parent FL2, child FLE, origin xyz=0.0 1.04 0.0 rpy=0.0 0.0 0.0
- added joint FREJ: type fixed, parent FR2, child FRE, origin xyz=0.0 1.04 0.0 rpy=0.0 0.0 0.0

Commit message: Fixed scale of urdf

File: urdfs/spider_bot_v0.urdf (robot description, URDF)
Before this commit: robot spiderbot, 17 links, 16 joints
Links:
- added link Servo0, mass 0.0134; collision box size=0.0228 0.0122 0.0285; visual box size=0.0228 0.0122 0.0285
- link BL0: geometry collision box size=0.03683 0.043134 0.0127; visual box size=0.03683 0.043134 0.0127
- link BL1: geometry collision box size=0.0127 0.06541 0.0381; visual box size=0.0127 0.06541 0.0381
- link BL2: geometry collision cylinder length=0.104 radius=.008; visual cylinder length=0.104 radius=.008
- link BLE: geometry collision sphere radius=0.008; visual sphere radius=0.008
- link BR0: geometry collision box size=0.03683 0.043134 0.0127; visual box size=0.03683 0.043134 0.0127
- link BR1: geometry collision box size=0.0127 0.06541 0.0381; visual box size=0.0127 0.06541 0.0381
- link BR2: geometry collision cylinder length=0.104 radius=.008; visual cylinder length=0.104 radius=.008
- link BRE: geometry collision sphere radius=0.008; visual sphere radius=0.008
- link FL0: geometry collision box size=0.03683 0.043134 0.0127; visual box size=0.03683 0.043134 0.0127
- link FL1: geometry collision box size=0.0127 0.06541 0.0381; visual box size=0.0127 0.06541 0.0381
- link FL2: geometry collision cylinder length=0.104 radius=.008; visual cylinder length=0.104 radius=.008
- link FLE: geometry collision sphere radius=0.008; visual sphere radius=0.008
- link FR0: geometry collision box size=0.03683 0.043134 0.0127; visual box size=0.03683 0.043134 0.0127
- link FR1: geometry collision box size=0.0127 0.06541 0.0381; visual box size=0.0127 0.06541 0.0381
- link FR2: geometry collision cylinder length=0.104 radius=.008; visual cylinder length=0.104 radius=.008
- link FRE: geometry collision sphere radius=0.008; visual sphere radius=0.008
- link SpiderBody: geometry collision box size=0.095 0.093 0.089; visual box size=0.095 0.093 0.089
Joints:
- added joint S0J: type fixed, parent SpiderBody, child Servo0, origin xyz=-0.034317 -0.048021 0 rpy=0.0 0.0 0.0
- joint BLEJ: origin xyz=0.0 1.04 0.0 rpy=0.0 0.0 0.0 -> xyz=0.0 0.104 0.0 rpy=0.0 0.0 0.0
- joint BLJ0: origin xyz=0.34317 -0.50021 0 rpy=0.0 0 3.1415 -> xyz=0.034317 -0.050021 0 rpy=0.0 0 3.1415
- joint BLJ1: origin xyz=0 0.28395 0 rpy=0 0 0 -> xyz=0 0.028395 0 rpy=0 0 0
- joint BLJ2: origin xyz=0 0.6 0 rpy=0 0 0 -> xyz=0 0.06 0 rpy=0 0 0
- joint BREJ: origin xyz=0.0 1.04 0.0 rpy=0.0 0.0 0.0 -> xyz=0.0 0.104 0.0 rpy=0.0 0.0 0.0
- joint BRJ0: origin xyz=0.34317 0.50021 0 rpy=0.0 0 0 -> xyz=0.034317 0.050021 0 rpy=0.0 0 0
- joint BRJ1: origin xyz=0 0.28395 0 rpy=0 0 0 -> xyz=0 0.028395 0 rpy=0 0 0
- joint BRJ2: origin xyz=0 0.6 0 rpy=0 0 0 -> xyz=0 0.06 0 rpy=0 0 0
- joint FLEJ: origin xyz=0.0 1.04 0.0 rpy=0.0 0.0 0.0 -> xyz=0.0 0.104 0.0 rpy=0.0 0.0 0.0
- joint FLJ0: origin xyz=-0.34317 -0.50021 0 rpy=0.0 0 3.1415 -> xyz=-0.034317 -0.050021 0 rpy=0.0 0 3.1415
- joint FLJ1: origin xyz=0 0.28395 0 rpy=0 0 0 -> xyz=0 0.028395 0 rpy=0 0 0
- joint FLJ2: origin xyz=0 0.6 0 rpy=0 0 0 -> xyz=0 0.06 0 rpy=0 0 0
- joint FREJ: origin xyz=0.0 1.04 0.0 rpy=0.0 0.0 0.0 -> xyz=0.0 0.104 0.0 rpy=0.0 0.0 0.0
- joint FRJ0: origin xyz=-0.34317 0.50021 0 rpy=0.0 0 0 -> xyz=-0.034317 0.050021 0 rpy=0.0 0 0
- joint FRJ1: origin xyz=0 0.28395 0 rpy=0 0 0 -> xyz=0 0.028395 0 rpy=0 0 0
- joint FRJ2: origin xyz=0 0.6 0 rpy=0 0 0 -> xyz=0 0.06 0 rpy=0 0 0
