Commit message: Adjusted mass to be accurate with urdf units. Still need to adjust inertia matrix and the referance position

File: urdfs/spider_bot_v2.urdf (robot description, URDF)
Before this commit: robot spiderbot, 18 links, 17 joints
Links:
- added link Servo1, mass 0.0134; collision box size=0.0228 0.0122 0.0285; visual box size=0.0228 0.0122 0.0285
- added link Servo10, mass 0.0134; collision box size=0.0228 0.0122 0.0285; visual box size=0.0228 0.0122 0.0285
- added link Servo11, mass 0.0134; collision box size=0.0228 0.0122 0.0285; visual box size=0.0228 0.0122 0.0285
- added link Servo2, mass 0.0134; collision box size=0.0228 0.0122 0.0285; visual box size=0.0228 0.0122 0.0285
- added link Servo3, mass 0.0134; collision box size=0.0228 0.0122 0.0285; visual box size=0.0228 0.0122 0.0285
- added link Servo4, mass 0.0134; collision box size=0.0228 0.0122 0.0285; visual box size=0.0228 0.0122 0.0285
- added link Servo5, mass 0.0134; collision box size=0.0228 0.0122 0.0285; visual box size=0.0228 0.0122 0.0285
- added link Servo6, mass 0.0134; collision box size=0.0228 0.0122 0.0285; visual box size=0.0228 0.0122 0.0285
- added link Servo7, mass 0.0134; collision box size=0.0228 0.0122 0.0285; visual box size=0.0228 0.0122 0.0285
- added link Servo8, mass 0.0134; collision box size=0.0228 0.0122 0.0285; visual box size=0.0228 0.0122 0.0285
- added link Servo9, mass 0.0134; collision box size=0.0228 0.0122 0.0285; visual box size=0.0228 0.0122 0.0285
- link BL0: mass 1 -> 0.005
- link BL1: mass 1 -> 0.005
- link BL2: mass 1 -> 0.005
- link BLE: mass 0.5 -> 0.001
- link BR0: mass 1 -> 0.005
- link BR1: mass 1 -> 0.005
- link BR2: mass 1 -> 0.005
- link BRE: mass 0.5 -> 0.001
- link FL0: mass 1 -> 0.005
- link FL1: mass 1 -> 0.005
- link FL2: mass 1 -> 0.005
- link FLE: mass 0.5 -> 0.001
- link FR0: mass 1 -> 0.005
- link FR1: mass 1 -> 0.005
- link FR2: mass 1 -> 0.005
- link FRE: mass 0.5 -> 0.001
- link SpiderBody: mass 25 -> 0.8184311
Joints:
- added joint S10J: type fixed, parent BR2, child Servo10, origin xyz=0 0 0 rpy=1.571 1.571 0.0
- added joint S11J: type fixed, parent FR2, child Servo11, origin xyz=0 0 0 rpy=1.571 1.571 0.0
- added joint S1J: type fixed, parent SpiderBody, child Servo1, origin xyz=0.036 -0.045021 0 rpy=0.0 0.0 0.0
- added joint S2J: type fixed, parent SpiderBody, child Servo2, origin xyz=0.036 0.045021 0 rpy=0.0 0.0 0.0
- added joint S3J: type fixed, parent SpiderBody, child Servo3, origin xyz=-0.032 0.045021 0 rpy=0.0 0.0 0.0
- added joint S4J: type fixed, parent FL0, child Servo4, origin xyz=0 0.028395 0 rpy=0.0 1.571 0.0
- added joint S5J: type fixed, parent BL0, child Servo5, origin xyz=0 0.028395 0 rpy=0.0 1.571 0.0
- added joint S6J: type fixed, parent BR0, child Servo6, origin xyz=0 0.028395 0 rpy=0.0 1.571 0.0
- added joint S7J: type fixed, parent FR0, child Servo7, origin xyz=0 0.028395 0 rpy=0.0 1.571 0.0
- added joint S8J: type fixed, parent FL2, child Servo8, origin xyz=0 0 0 rpy=1.571 1.571 0.0
- added joint S9J: type fixed, parent BL2, child Servo9, origin xyz=0 0 0 rpy=1.571 1.571 0.0
- joint S0J: origin xyz=-0.034317 -0.048021 0 rpy=0.0 0.0 0.0 -> xyz=-0.032 -0.045021 0 rpy=0.0 0.0 0.0

Commit message: improved multiprocessing and assertions

File: urdfs/spider_bot_v2.urdf (robot description, URDF)
Before this commit: robot spiderbot, 29 links, 28 joints
Links:
- removed link Servo0
- removed link Servo1
- removed link Servo10
- removed link Servo11
- removed link Servo2
- removed link Servo3
- removed link Servo4
- removed link Servo5
- removed link Servo6
- removed link Servo7
- removed link Servo8
- removed link Servo9
Joints:
- removed joint S0J
- removed joint S10J
- removed joint S11J
- removed joint S1J
- removed joint S2J
- removed joint S3J
- removed joint S4J
- removed joint S5J
- removed joint S6J
- removed joint S7J
- removed joint S8J
- removed joint S9J

Commit message: tools to help debug joint pos errors

File: urdfs/spider_bot_v2.urdf (robot description, URDF)
Before this commit: robot spiderbot, 17 links, 16 joints
Joints:
- joint BLEJ: limit (none) -> lower=-1.0 upper=0.0 effort=100 velocity=100
- joint BREJ: limit (none) -> lower=-1.0 upper=0.0 effort=100 velocity=100
- joint FLEJ: limit (none) -> lower=-1.0 upper=0.0 effort=100 velocity=100
- joint FREJ: limit (none) -> lower=-1.0 upper=0.0 effort=100 velocity=100
